File: KICAD/DCU.kicad_pcb (KiCad board)
At the start: 2 copper layers, 65 x 70 mm, 116 parts, among them J1 Conn_01x10_Female, J2 Conn_01x06_Female, J3 Conn_01x04_Male, J4 Conn_01x04_Female, J5 Conn_01x04_Female, J6 ARM_JTAG_SWD_10, U1 LM358, U2 SN65HVD233, U3 ADP150AUJZ-3.3-R7, U4 LM358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

Commit message: test
Other:
- net class Default removed
- net class Power removed
