File: KICAD/DCU.kicad_sch (KiCad schematic)
At the start: 5 parts, among them J1 Conn_01x10_Female, J2 Conn_01x06_Female, J3 Conn_01x04_Male, J4 Conn_01x04_Female, J5 Conn_01x04_Female

Commit message: Name change
Other:
- title: DRIVER CONTROL UNIT (DCU) -> VEHICLE MEASUREMENT UNIT (VMU)
