File: KICAD/MCU.kicad_sch (KiCad schematic)
At the start: 24 parts, among them J6 ARM_JTAG_SWD_10, U2 SN65HVD233, U7 STM32F091RCTx

Commit message: Changed name on MCU
Connections:
- net +3.3V: no longer J6.1 (VTref)
- net +5V: no longer D29.2 (K)
- net GND: no longer D29.1 (A), J6.3 (GND), J6.5 (GND), J6.9 (GNDDetect)
- net JTAG_RESET_N: no longer J6.10 (~{RESET})
- net JTAG_SWDCLK: no longer J6.4 (SWDCLK/TCK)
- net JTAG_SWDIO: no longer J6.2 (SWDIO/TMS)
- net at R?.1: no longer D29.3 (common)
- net at R?.2: no longer D29.3 (common)
Other:
- title: DRIVER CONTROL UNIT (DCU) -> VMU (VEHICLE MEASUREMENT UNIT)

Commit message: Name change
Other:
- title: VMU (VEHICLE MEASUREMENT UNIT) -> VEHICLE MEASUREMENT UNIT (VMU)
