File: KICAD/POWER.kicad_sch (KiCad schematic)
At the start: 26 parts, among them U3 ADP150AUJZ-3.3-R7

Commit message: Changed name on MCU
Connections:
- net +24V: no longer VR1.1 (IN)
- net +3.3V: no longer U3.5 (VOUT)
- net +5V: no longer U3.1 (VIN), U3.3 (EN)
- net GND: no longer U3.2 (GND), VR1.2 (GND)

Commit message: Updated power and changed name
Updated the power sch and changed the name of the MCU.
Other:
- title: DRIVER CONTROL UNIT (DCU) -> VEHICLE MEASUREMENT UNIT (VMU)
